Commit message: Added RGBD Camera configuration

File: src/my_robot/urdf/my_robot.xacro (robot description, xacro)
@@ -193,3 +193,11 @@
     <material>Gazebo/Orange</material>
 </gazebo>
+<!-- Optical Camera Link -->
+<joint name="camera_optical_joint" type="fixed">
+  <origin xyz="0 0 0" rpy="-1.5707 0 -1.5707"/>
+  <parent link="camera_link"/>
+  <child link="camera_link_optical"/>
+</joint>
+<link name="camera_link_optical">
+</link>
 </robot>

Commit message: Working on bug  Not resolved

File: src/my_robot/urdf/my_robot.xacro (robot description, xacro)
@@ -196,5 +196,5 @@
 <joint name="camera_optical_joint" type="fixed">
   <origin xyz="0 0 0" rpy="-1.5707 0 -1.5707"/>
-  <parent link="camera_link"/>
+  <parent link="camera"/>
   <child link="camera_link_optical"/>
 </joint>

Commit message: Links work. New bug: Grid map is empty, Large map

File: src/my_robot/urdf/my_robot.xacro (robot description, xacro)
@@ -122,5 +122,40 @@
     <inertial>
       <origin xyz="0 0 0" rpy="0 0 0"/>
+      <geometry>
+        <box size="0.05 0.05 0.05"/>
+      </geometry>
       <mass value="0.1"/>
+      <inertia
+	       ixx="1e-6" ixy="0" ixz="0"
+	       iyy="1e-6" iyz="0"
+	       izz="1e-6"/>
+    </inertial>
+    <visual>
+	     <origin xyz="0 0 0" rpy="0 0 0" />
+       <geometry>
+        <box size="0.05 0.05 0.05" />
+      </geometry>
+    </visual>
+    <collision>
+	     <origin xyz="0 0 0" rpy="0 0 0" />
+        <geometry>
+	         <box size="0.05 0.05 0.05"/>
+	      </geometry>
+    </collision>
+  </link>
+<!--Add a joint of Camera-->
+ <joint type="fixed" name="camera_joint">
+    <origin xyz="0.2 0 0" rpy="0 0 0"/>
+    <child link="camera"/>
+    <parent link="chassis"/>
+    <!--<axis xyz="0 1.0 0" rpy="0 0 0"/>
+    <limit effort="10000" velocity="1000"/>
+    <dynamics damping="1.0" friction="1.0"/>-->
+  </joint>
+<!--Add a Lidar-->
+<link name="hokuyo">
+    <inertial>
+      <origin xyz="0 0 0" rpy="0 0 0"/>
+      <mass value="1e-5"/>
       <inertia
 	       ixx="1e-6" ixy="0" ixz="0"
@@ -130,37 +165,4 @@
     </inertial>
     <visual>
-	<origin xyz="0 0 0" rpy="0 0 0" />
-        <geometry>
-	<box size="0.05 0.05 0.05"/>
-	</geometry>
-    </visual>
-    <collision>
-	<origin xyz="0 0 0" rpy="0 0 0" />
-        <geometry>
-	<box size="0.05 0.05 0.05"/>
-	</geometry>
-    </collision>
-  </link>
-<!--Add a joint of Camera-->
- <joint type="fixed" name="camera_joint">
-    <origin xyz="0.2 0 0" rpy="0 0 0"/>
-    <child link="camera"/>
-    <parent link="chassis"/>
-    <axis xyz="0 1.0 0" rpy="0 0 0"/>
-    <limit effort="10000" velocity="1000"/>
-    <dynamics damping="1.0" friction="1.0"/>
-  </joint>
-<!--Add a Lidar-->
-<link name="hokuyo">
-    <inertial>
-      <origin xyz="0 0 0" rpy="0 0 0"/>
-      <mass value="1e-5"/>
-      <inertia
-	       ixx="1e-6" ixy="0" ixz="0"
-	       iyy="1e-6" iyz="0"
-	       izz="1e-6"
-	/>
-    </inertial>
-    <visual>
       <origin xyz="0 0 0" rpy="0 0 0"/>
       <geometry>
@@ -180,7 +182,7 @@
     <child link="hokuyo"/>
     <parent link="chassis"/>
-    <axis xyz="0 1.0 0" rpy="0 0 0"/>
-    <limit effort="10000" velocity="1000"/>
-    <dynamics damping="1.0" friction="1.0"/>
+  <!--  <axis xyz="0 1.0 0" rpy="0 0 0"/>
+    <limit effort="10000" velocity="1000"/>
+    <dynamics damping="1.0" friction="1.0"/>-->
   </joint>
 <gazebo reference="left_wheel">
@@ -192,4 +194,7 @@
 <gazebo reference="chassis">
     <material>Gazebo/Orange</material>
+</gazebo>
+<gazebo reference="camera">
+    <material>Gazebo/Blue</material>
 </gazebo>
 <!-- Optical Camera Link -->
